File: Hardware/dc32.kicad_sch (KiCad schematic)
At the start: 48 parts, among them J2 Conn_01x50, J2 Micro_SD_Card_SPI, SW14 SW_SPDT, SW7 Function Select, U1 Pico, U2 INMP4441, U3 MAX98357A/B, U4 SC189ZULTRT, X1 Badgelife_sao_connector_v169b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

Commit message: Cleaning schematic, ERC, making sure all footprints are in place
Parts:
- added H1: Top Right, MountingHole:MountingHole_3.2mm_M3_Pad_Via, symbol Mechanical:MountingHole_Pad
- added H2: Top Left, MountingHole:MountingHole_3.2mm_M3_Pad_Via, symbol Mechanical:MountingHole_Pad
- added H3: Bottom Right, MountingHole:MountingHole_3.2mm_M3_Pad_Via, symbol Mechanical:MountingHole_Pad
- added H4: Bottom Left, MountingHole:MountingHole_3.2mm_M3_Pad_Via, symbol Mechanical:MountingHole_Pad
- added X2: Badgelife_sao_connector_v169bis, lib_fp:Badgelife-Shitty-v1.69bis-Minimal-Front, symbol badgelife_shitty_addon_v169bis:Badgelife_sao_connector_v169bis
- D19: renamed from D15; footprint Diode_SMD:D_SOD-323 -> Diode_SMD:D_SOD-523
- U2: footprint (none) -> lib_fp:MIC_INMP441ACEZ-R7
- renumbered C3 to C1, C1 to C4, C6 to C5, C5 to C6, D16 to D14, D17 to D15, D18 to D16, D19 to D17, D20 to D18, FID3 to FID1, FID4 to FID3, FID1 to FID4, R2 to R1, R1 to R2, R7 to R4, SW14 to SW1, TP2 to TP1, TP3 to TP2, TP1 to TP3, U4 to U1, U1 to U3, U3 to U4
Connections:
- net +3V3: now also H1.1, X2.1 (VCC)
- net ENC1_SW: now also U3.25 (GPIO19)
- net GND: now also H4.1, X2.2 (GND)
- net SCL: no longer X1.4 (SCL)
- net SDA: no longer X1.3 (SDA)
- net at TP4.1: now also U4.10 (OUTN); no longer U4.9 (OUTP)
- net at TP5.1: now also U4.9 (OUTP); no longer U4.10 (OUTN)
- no-connect marks 29 -> 37
Other:
- moved on the sheet: FID1, FID2, FID3, FID4, SW7, TP4, TP5, X1

Commit message: Updated PCBs to rev 1.0 and ordered them
Parts:
- removed X1, X2: Badgelife_sao_connector_v169bis, lib_fp:Badgelife-Shitty-v1.69bis-Minimal-Front, symbol badgelife_shitty_addon_v169bis:Badgelife_sao_connector_v169bis
- U1: footprint lib_fp:SC189ZULTRT -> Package_TO_SOT_SMD:SOT-23-5
Connections:
- net SDA is gone; now on net RGB: U3.19 (GPIO14)
- net +3V3: now also U1.4 (OUT); no longer U1.6 (OUT)
- net GND: now also U1.2 (GND); no longer U1.5 (GND)
- net RGB: no longer U3.24 (GPIO18)
- net VCC: now also U1.1 (Vin); no longer U1.2 (EN)
- net at L1.1: now also U1.5 (LX); no longer U1.4 (LX)
- net SCL: no longer names the net of U3.20 (GPIO15)
- no-connect marks 37 -> 29
